File: dronestand.brd (EAGLE design)
At the start: 62.2 x 65.7 mm, 14 parts, among them Q1 FDD4141TO252, Q5 FDD4141TO252

Commit message: Second commit of drone stand control board
Parts:
- added POT: (no value), pinhead:1X03
Connections:
- new net SIGNAL: ARDUINO_NANO1.9, POT.2
- net GND/VCC: now also POT.3
- net VCC: now also POT.1
Routing:
- net SIGNAL: track 0.00 -> 45.6 mm
- net VCC: track 93.5 -> 108.3 mm
Changed lines of the file:
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@@
 <attribute name="VALUE" x="11.6856" y="71.1526" size="0.9906" layer="27" ratio="10" rot="R180"/>
+</element>
+<element name="POT" library="pinhead" library_urn="urn:adsk.eagle:library:325" package="1X03" package3d_urn="urn:adsk.eagle:package:22458/2" value="" x="8.9" y="25.4" smashed="yes">
+<attribute name="NAME" x="5.0138" y="27.2288" size="1.27" layer="25" ratio="10"/>
+<attribute name="VALUE" x="5.09" y="22.225" size="1.27" layer="27"/>
 </element>
 </elements>
@@
 <wire x1="11.63" y1="49.18" x2="15.79" y2="53.34" width="0.8128" layer="16"/>
 <wire x1="15.79" y1="53.34" x2="17.78" y2="53.34" width="0.8128" layer="16"/>
+<contactref element="POT" pad="3"/>
 </signal>
 <signal name="5V">
@@
 <wire x1="10.1" y1="72.9" x2="7.87" y2="70.67" width="1.27" layer="1"/>
 <wire x1="7.87" y1="70.67" x2="6.25" y2="70.67" width="1.27" layer="1"/>
+<contactref element="POT" pad="1"/>
+<wire x1="6.36" y1="25.4" x2="3.5" y2="28.26" width="1.27" layer="1"/>
+<wire x1="3.5" y1="28.26" x2="3.5" y2="35" width="1.27" layer="1"/>
+<wire x1="3.5" y1="35" x2="5.1" y2="36.6" width="1.27" layer="1"/>
+<wire x1="5.1" y1="36.6" x2="6.8" y2="36.6" width="1.27" layer="1"/>
+<wire x1="6.8" y1="36.6" x2="6.25" y2="36.43" width="0" layer="19" extent="1-1"/>
 </signal>
 <signal name="NPN1">
@@
 <via x="55.1" y="47.3" extent="1-16" drill="1"/>
 </signal>
+<signal name="SIGNAL">
+<contactref element="POT" pad="2"/>
+<contactref element="ARDUINO_NANO1" pad="9"/>
+<wire x1="8.9" y1="25.4" x2="11.1" y2="23.2" width="1.27" layer="16"/>
+<wire x1="11.1" y1="23.2" x2="19.2" y2="23.2" width="1.27" layer="16"/>
+<wire x1="19.2" y1="23.2" x2="26.2" y2="30.2" width="1.27" layer="16"/>
+<wire x1="26.2" y1="50" x2="22.86" y2="53.34" width="1.27" layer="16"/>
+<wire x1="26.2" y1="30.2" x2="26.2" y2="50" width="1.27" layer="16"/>
+</signal>
 </signals>
