File: dronestand.sch (EAGLE design)
At the start: 14 parts, among them Q1 FDD4141TO252, Q5 FDD4141TO252

Commit message: Second commit of drone stand control board
Parts:
- added POT: (no value), pinhead:PINHD-1X3
Connections:
- new net SIGNAL: ARDUINO_NANO1.A5, POT.2
- net GND/VCC: now also POT.3
- net VCC: now also POT.1
Changed lines of the file:
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@@
 <setting verticaltext="up"/>
 </settings>
-<grid distance="0.1" unitdist="inch" unit="inch" style="lines" multiple="1" display="no" altdistance="0.01" altunitdist="inch" altunit="inch"/>
+<grid distance="0.1" unitdist="mm" unit="mm" style="lines" multiple="1" display="no" altdistance="0.1" altunitdist="mm" altunit="mm"/>
 <layers>
 <layer number="1" name="Top" color="4" fill="1" visible="no" active="no"/>
@@
 <part name="Q5" library="transistor-fet" library_urn="urn:adsk.eagle:library:396" deviceset="FDD4141" device="TO252" package3d_urn="urn:adsk.eagle:package:28537/2"/>
 <part name="Q1" library="transistor-fet" library_urn="urn:adsk.eagle:library:396" deviceset="FDD4141" device="TO252" package3d_urn="urn:adsk.eagle:package:28537/2"/>
+<part name="POT" library="pinhead" library_urn="urn:adsk.eagle:library:325" deviceset="PINHD-1X3" device="" package3d_urn="urn:adsk.eagle:package:22458/2"/>
 </parts>
 <sheets>
@@
 <attribute name="VALUE" x="-157.48" y="53.34" size="1.778" layer="96"/>
 <attribute name="NAME" x="-157.48" y="55.88" size="1.778" layer="95"/>
+</instance>
+<instance part="POT" gate="A" x="-246.38" y="81.28" smashed="yes" rot="R180">
+<attribute name="NAME" x="-240.03" y="75.565" size="1.778" layer="95" rot="R180"/>
+<attribute name="VALUE" x="-240.03" y="88.9" size="1.778" layer="96" rot="R180"/>
 </instance>
 </instances>
@@
 <junction x="-30.48" y="134.62"/>
 </segment>
+<segment>
+<pinref part="POT" gate="A" pin="1"/>
+<wire x1="-243.84" y1="78.74" x2="-236.22" y2="78.74" width="0.1524" layer="91"/>
+<label x="-238.76" y="78.74" size="1.778" layer="95"/>
+</segment>
 </net>
 <net name="NPN1" class="0">
@@
 <pinref part="Q1" gate="G$1" pin="G"/>
 </segment>
+<segment>
+<pinref part="POT" gate="A" pin="3"/>
+<wire x1="-243.84" y1="83.82" x2="-236.22" y2="83.82" width="0.1524" layer="91"/>
+<label x="-238.76" y="83.82" size="1.778" layer="95"/>
+</segment>
 </net>
 <net name="INT" class="0">
@@
 </segment>
 </net>
+<net name="SIGNAL" class="0">
+<segment>
+<pinref part="POT" gate="A" pin="2"/>
+<wire x1="-243.84" y1="81.28" x2="-236.22" y2="81.28" width="0.1524" layer="91"/>
+<label x="-238.76" y="81.28" size="1.778" layer="95"/>
+</segment>
+<segment>
+<pinref part="ARDUINO_NANO1" gate="G$1" pin="A5"/>
+<wire x1="-160.02" y1="123.19" x2="-154.94" y2="123.19" width="0.1524" layer="91"/>
+<label x="-157.5" y="123.4" size="1.778" layer="95"/>
+</segment>
+</net>
